File: Alfond_PCB/_autosave-Alfond PCB.kicad_sch (KiCad schematic)
At the start: 47 parts, among them J1 Micro_SD_Card_Det_Hirose_DM3AT, J2 USB_B_Micro, J3 Conn_01x04_Pin, SW1 SW_SPDT, U1 STM32U535VCT6, U2 DS18B20, U3 MS8607-02BA01, U5 MIC5219-3.3YMM, Y1 16MHz

Commit message: copy with the stm32u535
Other:
- note added: "look into vcap"
Changed lines of the file:
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@@
+		)
+	)
+	(text "look into vcap\n"
+		(exclude_from_sim no)
+		(at 158.75 164.338 0)
+		(effects
+			(font
+				(size 1.27 1.27)
+			)
 		)
 	)
