File: Alfond_PCB/Alfond PCB.kicad_sch (KiCad schematic)
At the start: 47 parts, among them J1 Micro_SD_Card_Det_Hirose_DM3AT, J2 USB_B_Micro, J3 Conn_01x04_Pin, SW1 SW_SPDT, U1 STM32U535VCT6, U2 DS18B20, U3 MS8607-02BA01, U5 MIC5219-3.3YMM, Y1 16MHz

Commit message: saved copy with the stm32u535
Connections:
- net HSE_OUT is gone; now on net HSE_IN: C15.1, U1.13 (PH1), Y1.1
Other:
- note added: "look into vcap"
Changed lines of the file:
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@@
+	)
+	(junction
+		(at 167.64 120.65)
+		(diameter 0)
+		(color 0 0 0 0)
 	)
 	(junction
@@
 	)
 	(junction
+		(at 166.37 67.31)
+		(diameter 0)
+		(color 0 0 0 0)
+	)
+	(junction
 		(at 82.55 41.91)
 		(diameter 0)
@@
 	)
 	(junction
+		(at 165.1 67.31)
+		(diameter 0)
+		(color 0 0 0 0)
+	)
+	(junction
 		(at 92.71 34.29)
 		(diameter 0)
@@
 	)
 	(junction
+		(at 165.1 64.77)
+		(diameter 0)
+		(color 0 0 0 0)
+	)
+	(junction
+		(at 214.63 107.95)
+		(diameter 0)
+		(color 0 0 0 0)
+	)
+	(junction
 		(at 125.73 26.67)
 		(diameter 0)
@@
 	(wire
 		(pts
+			(xy 166.37 67.31) (xy 177.8 67.31)
+		)
+		(stroke
+			(width 0)
+			(type default)
+		)
+	)
+	(wire
+		(pts
 			(xy 156.21 69.85) (xy 162.56 69.85)
 		)
@@
 	(wire
 		(pts
-			(xy 156.21 64.77) (xy 204.47 64.77)
+			(xy 156.21 64.77) (xy 165.1 64.77)
 		)
 		(stroke
@@
 	(wire
 		(pts
+			(xy 212.09 110.49) (xy 214.63 110.49)
+		)
+		(stroke
+			(width 0)
+			(type default)
+		)
+	)
+	(wire
+		(pts
 			(xy 104.14 82.55) (xy 110.49 82.55)
 		)
@@
 	(wire
 		(pts
+			(xy 99.06 77.47) (xy 110.49 77.47)
+		)
+		(stroke
+			(width 0)
+			(type default)
+		)
+	)
+	(wire
+		(pts
 			(xy 172.72 39.37) (xy 187.96 39.37)
 		)
@@
 	(wire
 		(pts
-			(xy 99.06 77.47) (xy 110.49 77.47)
-		)
-		(stroke
-			(width 0)
-			(type default)
-		)
-	)
-	(wire
-		(pts
 			(xy 48.26 129.54) (xy 60.96 129.54)
 		)
@@
 	(wire
 		(pts
+			(xy 166.37 123.19) (xy 167.64 123.19)
+		)
+		(stroke
+			(width 0)
+			(type default)
+		)
+	)
+	(wire
+		(pts
 			(xy 44.45 48.26) (xy 48.26 48.26)
 		)
@@
 	(wire
 		(pts
-			(xy 210.82 107.95) (xy 217.17 107.95)
-		)
-		(stroke
-			(width 0)
-			(type default)
-		)
-	)
-	(wire
-		(pts
 			(xy 270.51 86.36) (xy 267.97 86.36)
 		)
@@
 	(wire
 		(pts
-			(xy 156.21 67.31) (xy 177.8 67.31)
+			(xy 214.63 107.95) (xy 217.17 107.95)
+		)
+		(stroke
+			(width 0)
+			(type default)
+		)
+	)
+	(wire
+		(pts
+			(xy 214.63 110.49) (xy 214.63 107.95)
+		)
+		(stroke
+			(width 0)
+			(type default)
+		)
+	)
+	(wire
+		(pts
+			(xy 156.21 67.31) (xy 165.1 67.31)
 		)
 		(stroke
@@
 	(wire
 		(pts
-			(xy 156.21 120.65) (xy 173.99 120.65)
-		)
-		(stroke
-			(width 0)
-			(type default)
-		)
-	)
-	(wire
-		(pts
 			(xy 82.55 41.91) (xy 92.71 41.91)
 		)
@@
 	(wire
 		(pts
+			(xy 210.82 107.95) (xy 214.63 107.95)
+		)
+		(stroke
+			(width 0)
+			(type default)
+		)
+	)
+	(wire
+		(pts
 			(xy 130.81 40.64) (xy 130.81 44.45)
 		)
@@
 	(wire
 		(pts
+			(xy 165.1 67.31) (xy 165.1 64.77)
+		)
+		(stroke
+			(width 0)
+			(type default)
+		)
+	)
+	(wire
+		(pts
 			(xy 214.63 78.74) (xy 232.41 78.74)
 		)
@@
 	(wire
 		(pts
+			(xy 187.96 57.15) (xy 190.5 57.15)
+		)
+		(stroke
+			(width 0)
+			(type default)
+		)
+	)
+	(wire
+		(pts
 			(xy 204.47 146.05) (xy 204.47 143.51)
 		)
@@
 	(wire
 		(pts
-			(xy 187.96 57.15) (xy 190.5 57.15)
+			(xy 165.1 64.77) (xy 204.47 64.77)
 		)
 		(stroke
@@
 	(wire
 		(pts
+			(xy 167.64 123.19) (xy 167.64 120.65)
+		)
+		(stroke
+			(width 0)
+			(type default)
+		)
+	)
+	(wire
+		(pts
 			(xy 93.98 90.17) (xy 93.98 92.71)
 		)
@@
 	(wire
 		(pts
+			(xy 156.21 120.65) (xy 167.64 120.65)
+		)
+		(stroke
+			(width 0)
+			(type default)
+		)
+	)
+	(wire
+		(pts
 			(xy 48.26 48.26) (xy 48.26 50.8)
 		)
@@
 	(wire
 		(pts
+			(xy 166.37 67.31) (xy 165.1 67.31)
+		)
+		(stroke
+			(width 0)
+			(type default)
+		)
+	)
+	(wire
+		(pts
+			(xy 167.64 120.65) (xy 173.99 120.65)
+		)
+		(stroke
+			(width 0)
+			(type default)
+		)
+	)
+	(wire
+		(pts
 			(xy 194.31 67.31) (xy 185.42 67.31)
 		)
@@
 		(pts
 			(xy 247.65 33.02) (xy 247.65 35.56)
+		)
+		(stroke
+			(width 0)
+			(type default)
+		)
+	)
+	(wire
+		(pts
+			(xy 166.37 69.85) (xy 166.37 67.31)
 		)
 		(stroke
@@
 		(effects
 			(font
+				(size 1.27 1.27)
+			)
+		)
+	)
+	(text "look into vcap\n"
+		(exclude_from_sim no)
+		(at 158.75 164.338 0)
+		(effects
+			(font
