File: Alfond_PCB/Alfond PCB.kicad_pcb (KiCad board)
At the start: 2 copper layers, 91.2 x 54.2 mm, 54 parts, among them J3 Conn_01x05_Pin, J5 USB_B_Micro, P1 PHR-2, SW1 SW_SPDT, U2 STM32U545VETx, U5 MIC5219-3.3YM5-TR, Y1 16MHz

Commit message: made changes to switch placement
Parts:
- moved SW1 3.22 mm to (210.8, 47.0)
Routing:
- net Net-(SW1-B): track 17.8 -> 21.1 mm
- net GND: track 354.6 -> 357.9 mm
- net +3.3V: track 262.5 -> 265.8 mm
Changed lines of the file:
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@@
 	(footprint "Button_Switch_SMD:SW_SPDT_PCM12"
 		(layer "F.Cu")
-		(at 210.85 50.22 180)
+		(at 210.75 47 180)
 		(descr "Ultraminiature Surface Mount Slide Switch, right-angle, https://www.ckswitches.com/media/1424/pcm.pdf")
 		(property "Reference" "SW1"
@@
 	)
 	(segment
+		(start 213 52.5)
+		(end 215.5 55)
+		(width 0.2)
+		(layer "F.Cu")
+		(net 2)
+	)
+	(segment
 		(start 218.5 64.75)
 		(end 218.5 66.325)
@@
 	)
 	(segment
-		(start 213.1 51.65)
-		(end 213.1 52.6)
-		(width 0.2)
-		(layer "F.Cu")
-		(net 2)
-	)
-	(segment
 		(start 176.4625 90.0375)
 		(end 176.5 90)
@@
 	)
 	(segment
-		(start 213.1 52.6)
-		(end 215.5 55)
-		(width 0.2)
-		(layer "F.Cu")
-		(net 2)
-	)
-	(segment
 		(start 169.5 80.5)
 		(end 173.4 80.5)
@@
 	)
 	(segment
+		(start 213 48.43)
+		(end 213 52.5)
+		(width 0.2)
+		(layer "F.Cu")
+		(net 2)
+	)
+	(segment
 		(start 174 90.0375)
 		(end 176.4625 90.0375)
@@
 	)
 	(segment
-		(start 208.6 51.65)
-		(end 208.6 56.1675)
-		(width 0.2)
-		(layer "F.Cu")
-		(net 4)
-	)
-	(segment
 		(start 185.7125 88.7125)
 		(end 186 89)
@@
 	)
 	(segment
-		(start 208.6 56.1675)
-		(end 214.75 62.3175)
+		(start 219 83.4325)
+		(end 219 81.675)
 		(width 0.2)
 		(layer "F.Cu")
@@
 	)
 	(segment
-		(start 219 83.4325)
-		(end 219 81.675)
+		(start 185.262499 86.549999)
+		(end 185.7125 87)
 		(width 0.2)
 		(layer "F.Cu")
@@
 	)
 	(segment
-		(start 185.262499 86.549999)
-		(end 185.7125 87)
+		(start 208.5 56.0675)
+		(end 214.75 62.3175)
 		(width 0.2)
 		(layer "F.Cu")
@@
 	)
 	(segment
+		(start 214.75 62.3175)
+		(end 214.75 64.4625)
+		(width 0.2)
+		(layer "F.Cu")
+		(net 4)
+	)
+	(segment
 		(start 217.15741 70.5)
 		(end 217.828705 69.828705)
@@
 	)
 	(segment
-		(start 214.75 62.3175)
-		(end 214.75 64.4625)
-		(width 0.2)
-		(layer "F.Cu")
-		(net 4)
-	)
-	(segment
 		(start 230.421295 69.421295)
 		(end 230.84259 69)
@@
 	)
 	(segment
+		(start 208.5 48.43)
+		(end 208.5 56.0675)
+		(width 0.2)
+		(layer "F.Cu")
+		(net 4)
+	)
+	(segment
 		(start 218 66.325)
 		(end 216.1375 64.4625)
@@
 	)
 	(segment
-		(start 210.1 51.65)
-		(end 210.1 53.9)
-		(width 0.2)
-		(layer "F.Cu")
-		(net 39)
-	)
-	(segment
 		(start 220.0875 63)
 		(end 219.1 63)
@@
 		(width 0.2)
 		(layer "F.Cu")
+		(net 39)
+	)
+	(segment
+		(start 210 48.43)
+		(end 210 54)
+		(width 0.2)
+		(layer "F.Cu")
